Commit message: update

File: urdfs/panda.urdf (robot description, URDF)
Before this commit: robot panda_kinect, 16 links, 15 joints
Links:
- link ft_sensor_link: geometry collision mesh filename=package://holodemo/meshes/force_torque_sensor.stl; visual mesh filename=package://holodemo/meshes/force_torque_sensor.dae

Commit message: Add all files for display

File: urdfs/panda.urdf (robot description, URDF)
Before this commit: robot panda_kinect, 16 links, 15 joints
Links:
- link panda_hand: geometry collision mesh filename=package://holodemo/meshes/collision/hand.stl; visual mesh filename=package://holodemo/meshes/visual/hand.dae
- link panda_leftfinger: geometry collision mesh filename=package://holodemo/meshes/collision/finger.stl; visual mesh filename=package://holodemo/meshes/visual/finger.dae
- link panda_link0: geometry collision mesh filename=package://holodemo/meshes/collision/link0.stl; visual mesh filename=package://holodemo/meshes/visual/link0.dae
- link panda_link1: geometry collision mesh filename=package://holodemo/meshes/collision/link1.stl; visual mesh filename=package://holodemo/meshes/visual/link1.dae
- link panda_link2: geometry collision mesh filename=package://holodemo/meshes/collision/link2.stl; visual mesh filename=package://holodemo/meshes/visual/link2.dae
- link panda_link3: geometry collision mesh filename=package://holodemo/meshes/collision/link3.stl; visual mesh filename=package://holodemo/meshes/visual/link3.dae
- link panda_link4: geometry collision mesh filename=package://holodemo/meshes/collision/link4.stl; visual mesh filename=package://holodemo/meshes/visual/link4.dae
- link panda_link5: geometry collision mesh filename=package://holodemo/meshes/collision/link5.stl; visual mesh filename=package://holodemo/meshes/visual/link5.dae
- link panda_link6: geometry collision mesh filename=package://holodemo/meshes/collision/link6.stl; visual mesh filename=package://holodemo/meshes/visual/link6.dae
- link panda_link7: geometry collision mesh filename=package://holodemo/meshes/collision/link7.stl; visual mesh filename=package://holodemo/meshes/visual/link7.dae
- link panda_rightfinger: geometry collision mesh filename=package://holodemo/meshes/collision/finger.stl; visual mesh filename=package://holodemo/meshes/visual/finger.dae
